File: PCB/power.kicad_sch (KiCad schematic)
At the start: 24 parts, among them J2 SUR_SM02B-SURS-TF, SW1 SW_SPDT_PCM12, U2 TPS62162DSG, U3 BQ24075RGT

Commit message: Migrate KiCad to version 8.0
Parts:
- renumbered C7 to C4, C8 to C5, C5 to C6, C6 to C8, C4 to C9, R4 to R14, R9 to R16, R7 to R18, R8 to R19, R6 to R4, R10 to R6, R5 to R9, U3 to U2, U2 to U4
