File: PCB/sensor.kicad_sch (KiCad schematic)
At the start: 16 parts, among them J3 SUR_SM06B-SURS-TF, U4 BNO08X

Commit message: Migrate KiCad to version 8.0
Parts:
- renumbered C9 to C11, C11 to C12, C10 to C7, JP1 to JP3, R14 to R10, R16 to R11, R15 to R13, R18 to R15, R13 to R21, U4 to U3
