File: PCB/usb.kicad_sch (KiCad schematic)
At the start: 5 parts, among them J1 GT-USB-7010ASV

Commit message: Migrate KiCad to version 8.0
Parts:
- renumbered R3 to R2, R2 to R3, TP6 to TP3, TP6 to TP4
